Commit message: create simple model

File: bme_gazebo_basics/urdf/simple_model.urdf (robot description, URDF)
Before this commit: robot simple_model, 2 links, 1 joints
Joints:
- joint simple_model__link_1_JOINT_0: axis 0 -1  0 -> 0  0  1; origin xyz=0.08164 -0.20119  0.5 rpy=-1.5708  0      0 -> xyz=-0.00269 -0.28628  0 rpy=-1.5708  0      0; type revolute -> continuous
