Commit message: add wheels

File: bme_gazebo_basics/urdf/mogi_bot.xacro (robot description, xacro)
@@ -1,4 +1,5 @@
 <?xml version='1.0'?>
 <robot name="mogi_bot" xmlns:xacro="http://www.ros.org/wiki/xacro">
+  <!-- STEP 1 -->
   <link name="base_footprint"></link>
   <joint name="base_footprint_joint" type="fixed">
@@ -55,3 +56,66 @@
     </visual>
   </link>
+  <!-- STEP 2 -->
+  <joint type="continuous" name="left_wheel_joint">
+    <origin xyz="0 0.15 0" rpy="0 0 0"/>
+    <child link="left_wheel"/>
+    <parent link="base_link"/>
+    <axis xyz="0 1 0" rpy="0 0 0"/>
+    <limit effort="10000" velocity="1000"/>
+    <dynamics damping="1.0" friction="1.0"/>
+  </joint>
+  <link name='left_wheel'>
+    <inertial>
+      <mass value="5.0"/>
+      <origin xyz="0 0 0" rpy="0 1.5707 1.5707"/>
+      <inertia
+          ixx="0.1" ixy="0" ixz="0"
+          iyy="0.1" iyz="0"
+          izz="0.1"
+      />
+    </inertial>
+    <collision name='collision'>
+      <origin xyz="0 0 0" rpy="0 1.5707 1.5707"/>
+      <geometry>
+        <cylinder size=".1 .05"/>
+      </geometry>
+    </collision>
+    <visual name='left_wheel_visual'>
+      <origin xyz="0 0 0" rpy="0 1.5707 1.5707"/>
+      <geometry>
+        <cylinder size=".1 .05"/>
+      </geometry>
+    </visual>
+  </link>
+  <joint type="continuous" name="right_wheel_joint">
+    <origin xyz="0 -0.15 0" rpy="0 0 0"/>
+    <child link="right_wheel"/>
+    <parent link="base_link"/>
+    <axis xyz="0 1 0" rpy="0 0 0"/>
+    <limit effort="10000" velocity="1000"/>
+    <dynamics damping="1.0" friction="1.0"/>
+  </joint>
+  <link name='right_wheel'>
+    <inertial>
+      <mass value="5.0"/>
+      <origin xyz="0 0 0" rpy="0 1.5707 1.5707"/>
+      <inertia
+          ixx="0.1" ixy="0" ixz="0"
+          iyy="0.1" iyz="0"
+          izz="0.1"
+      />
+    </inertial>
+    <collision name='collision'>
+      <origin xyz="0 0 0" rpy="0 1.5707 1.5707"/>
+      <geometry>
+        <cylinder size=".1 .05"/>
+      </geometry>
+    </collision>
+    <visual name='right_wheel_visual'>
+      <origin xyz="0 0 0" rpy="0 1.5707 1.5707"/>
+      <geometry>
+        <cylinder size=".1 .05"/>
+      </geometry>
+    </visual>
+  </link>
 </robot>

Commit message: fix cylinder description

File: bme_gazebo_basics/urdf/mogi_bot.xacro (robot description, xacro)
@@ -109,5 +109,5 @@
       <origin xyz="0 0 0" rpy="0 1.5707 1.5707"/>
       <geometry>
-        <cylinder size=".1 .05"/>
+        <cylinder raduis=".1" length=".05"/>
       </geometry>
     </collision>
@@ -115,5 +115,5 @@
       <origin xyz="0 0 0" rpy="0 1.5707 1.5707"/>
       <geometry>
-        <cylinder size=".1 .05"/>
+        <cylinder raduis=".1" length=".05"/>
       </geometry>
     </visual>

Commit message: fix cylinder description 2

File: bme_gazebo_basics/urdf/mogi_bot.xacro (robot description, xacro)
@@ -78,5 +78,5 @@
       <origin xyz="0 0 0" rpy="0 1.5707 1.5707"/>
       <geometry>
-        <cylinder size=".1 .05"/>
+        <cylinder radius=".1" length=".05"/>
       </geometry>
     </collision>
@@ -84,5 +84,5 @@
       <origin xyz="0 0 0" rpy="0 1.5707 1.5707"/>
       <geometry>
-        <cylinder size=".1 .05"/>
+        <cylinder radius=".1" length=".05"/>
       </geometry>
     </visual>
@@ -109,5 +109,5 @@
       <origin xyz="0 0 0" rpy="0 1.5707 1.5707"/>
       <geometry>
-        <cylinder raduis=".1" length=".05"/>
+        <cylinder radius=".1" length=".05"/>
       </geometry>
     </collision>
@@ -115,5 +115,5 @@
       <origin xyz="0 0 0" rpy="0 1.5707 1.5707"/>
       <geometry>
-        <cylinder raduis=".1" length=".05"/>
+        <cylinder radius=".1" length=".05"/>
       </geometry>
     </visual>

Commit message: update xacro with colors and meshes

File: bme_gazebo_basics/urdf/mogi_bot.xacro (robot description, xacro)
@@ -1,7 +1,9 @@
 <?xml version='1.0'?>
 <robot name="mogi_bot" xmlns:xacro="http://www.ros.org/wiki/xacro">
-  <!-- STEP 3 -->
+  <!-- STEP 3 - Gazebo plugin -->
   <xacro:include filename="$(find bme_gazebo_basics)/urdf/mogi_bot.gazebo" />
-  <!-- STEP 1 -->
+  <!-- STEP 4 - RViz colors -->
+  <xacro:include filename="$(find bme_gazebo_basics)/urdf/materials.xacro" />
+  <!-- STEP 1 - Robot chassis -->
   <link name="base_footprint"></link>
   <joint name="base_footprint_joint" type="fixed">
@@ -30,6 +32,8 @@
       <origin xyz="0 0 0" rpy=" 0 0 0"/>
       <geometry>
-        <box size=".4 .2 .1"/>
+        <!--box size=".4 .2 .1"/-->
+        <mesh filename = "package://bme_gazebo_basics/meshes/mogi_bot.dae"/>
       </geometry>
+      <material name="orange"/>
     </visual>
     <collision name='rear_caster_collision'>
@@ -58,5 +62,5 @@
     </visual>
   </link>
-  <!-- STEP 2 -->
+  <!-- STEP 2 - Wheels -->
   <joint type="continuous" name="left_wheel_joint">
     <origin xyz="0 0.15 0" rpy="0 0 0"/>
@@ -86,6 +90,8 @@
       <origin xyz="0 0 0" rpy="0 1.5707 1.5707"/>
       <geometry>
-        <cylinder radius=".1" length=".05"/>
+        <!--cylinder radius=".1" length=".05"/-->
+        <mesh filename = "package://bme_gazebo_basics/meshes/wheel.dae"/>
       </geometry>
+      <material name="green"/>
     </visual>
   </link>
@@ -117,7 +123,19 @@
       <origin xyz="0 0 0" rpy="0 1.5707 1.5707"/>
       <geometry>
-        <cylinder radius=".1" length=".05"/>
+        <!--cylinder radius=".1" length=".05"/-->
+        <mesh filename = "package://bme_gazebo_basics/meshes/wheel.dae"/>
       </geometry>
+      <material name="green"/>
     </visual>
   </link>
+  <!-- STEP 4 - Gazebo colors -->
+  <!--gazebo reference="left_wheel">
+    <material>Gazebo/Green</material>
+  </gazebo>
+  <gazebo reference="right_wheel">
+    <material>Gazebo/Green</material>
+  </gazebo>
+  <gazebo reference="base_link">
+    <material>Gazebo/Orange</material>
+  </gazebo-->
 </robot>

Commit message: Revert "Starter branch"

File: bme_gazebo_basics/urdf/mogi_bot.xacro (robot description, xacro)
@@ -1,6 +1,9 @@
 <?xml version='1.0'?>
 <robot name="mogi_bot" xmlns:xacro="http://www.ros.org/wiki/xacro">
-  <xacro:include filename="$(find bme_gazebo_basics)/urdf/mogi_bot.gazebo" /> <!-- differenciálhajtás plugin leírás-->
-  <xacro:include filename="$(find bme_gazebo_basics)/urdf/materials.xacro" /> <!-- színekhez-->
+  <!-- STEP 3 - Gazebo plugin -->
+  <xacro:include filename="$(find bme_gazebo_basics)/urdf/mogi_bot.gazebo" />
+  <!-- STEP 4 - RViz colors -->
+  <xacro:include filename="$(find bme_gazebo_basics)/urdf/materials.xacro" />
+  <!-- STEP 1 - Robot chassis -->
   <link name="base_footprint"></link>
   <joint name="base_footprint_joint" type="fixed">
@@ -13,5 +16,5 @@
     <inertial>
       <mass value="15.0"/>
-      <origin xyz="0 0 0" rpy="0 0 0"/>
+      <origin xyz="0.0 0 0" rpy=" 0 0 0"/>
       <inertia
           ixx="0.1" ixy="0" ixz="0"
@@ -21,5 +24,5 @@
     </inertial>
     <collision name='collision'>
-      <origin xyz="0 0 0" rpy="0 0 0"/>
+      <origin xyz="0 0 0" rpy=" 0 0 0"/>
       <geometry>
         <box size=".4 .2 .1"/>
@@ -27,13 +30,13 @@
     </collision>
     <visual name='base_link_visual'>
-      <origin xyz="0 0 0" rpy="0 0 0"/>
+      <origin xyz="0 0 0" rpy=" 0 0 0"/>
       <geometry>
         <!--box size=".4 .2 .1"/-->
         <mesh filename = "package://bme_gazebo_basics/meshes/mogi_bot.dae"/>
       </geometry>
-      <material name="green"/>
+      <material name="orange"/>
     </visual>
     <collision name='rear_caster_collision'>
-      <origin xyz="-0.15 0 -0.05" rpy="0 0 0"/>
+      <origin xyz="-0.15 0 -0.05" rpy=" 0 0 0"/>
       <geometry>
         <sphere radius="0.0499"/>
@@ -41,5 +44,5 @@
     </collision>
     <visual name='rear_caster_visual'>
-      <origin xyz="-0.15 0 -0.05" rpy="0 0 0"/>
+      <origin xyz="-0.15 0 -0.05" rpy=" 0 0 0"/>
       <geometry>
         <sphere radius="0.05"/>
@@ -47,5 +50,5 @@
     </visual>
     <collision name='front_caster_collision'>
-      <origin xyz="0.15 0 -0.05" rpy="0 0 0"/>
+      <origin xyz="0.15 0 -0.05" rpy=" 0 0 0"/>
       <geometry>
         <sphere radius="0.0499"/>
@@ -53,5 +56,5 @@
     </collision>
     <visual name='front_caster_visual'>
-      <origin xyz="0.15 0 -0.05" rpy="0 0 0"/>
+      <origin xyz="0.15 0 -0.05" rpy=" 0 0 0"/>
       <geometry>
         <sphere radius="0.05"/>
@@ -59,10 +62,11 @@
     </visual>
   </link>
-    <joint type="continuous" name="left_wheel_joint">
+  <!-- STEP 2 - Wheels -->
+  <joint type="continuous" name="left_wheel_joint">
     <origin xyz="0 0.15 0" rpy="0 0 0"/>
     <child link="left_wheel"/>
     <parent link="base_link"/>
     <axis xyz="0 1 0" rpy="0 0 0"/>
-    <limit effort="10000" velocity="1000"/> <!-- effort: torque limit ...-->
+    <limit effort="10000" velocity="1000"/>
     <dynamics damping="1.0" friction="1.0"/>
   </joint>
@@ -86,6 +90,8 @@
       <origin xyz="0 0 0" rpy="0 1.5707 1.5707"/>
       <geometry>
+        <!--cylinder radius=".1" length=".05"/-->
         <mesh filename = "package://bme_gazebo_basics/meshes/wheel.dae"/>
       </geometry>
+      <material name="green"/>
     </visual>
   </link>
@@ -117,7 +123,19 @@
       <origin xyz="0 0 0" rpy="0 1.5707 1.5707"/>
       <geometry>
+        <!--cylinder radius=".1" length=".05"/-->
         <mesh filename = "package://bme_gazebo_basics/meshes/wheel.dae"/>
       </geometry>
+      <material name="green"/>
     </visual>
   </link>
+  <!-- STEP 4 - Gazebo colors -->
+  <!--gazebo reference="left_wheel">
+    <material>Gazebo/Green</material>
+  </gazebo>
+  <gazebo reference="right_wheel">
+    <material>Gazebo/Green</material>
+  </gazebo>
+  <gazebo reference="base_link">
+    <material>Gazebo/Orange</material>
+  </gazebo-->
 </robot>

File: bme_gazebo_basics/urdf/mogi_bot_skid_steer.xacro (robot description, xacro)
@@ -1,6 +1,9 @@
 <?xml version='1.0'?>
 <robot name="mogi_bot" xmlns:xacro="http://www.ros.org/wiki/xacro">
-  <xacro:include filename="$(find bme_gazebo_basics)/urdf/mogi_bot_skid_steer.gazebo" /> <!-- differenciálhajtás plugin leírás-->
-  <xacro:include filename="$(find bme_gazebo_basics)/urdf/materials.xacro" /> <!-- színekhez-->
+  <!-- STEP 3 - Gazebo plugin -->
+  <xacro:include filename="$(find bme_gazebo_basics)/urdf/mogi_bot_skid_steer.gazebo" />
+  <!-- STEP 4 - RViz colors -->
+  <xacro:include filename="$(find bme_gazebo_basics)/urdf/materials.xacro" />
+  <!-- STEP 1 - Robot chassis -->
   <link name="base_footprint"></link>
   <joint name="base_footprint_joint" type="fixed">
@@ -12,6 +15,6 @@
     <pose>0 0 0.1 0 0 0</pose>
     <inertial>
-      <mass value="15.0"/>
-      <origin xyz="0 0 0" rpy="0 0 0"/>
+      <mass value="5.0"/>
+      <origin xyz="0.0 0 0" rpy=" 0 0 0"/>
       <inertia
           ixx="0.1" ixy="0" ixz="0"
@@ -21,5 +24,5 @@
     </inertial>
     <collision name='collision'>
-      <origin xyz="0 0 0" rpy="0 0 0"/>
+      <origin xyz="0 0 0" rpy=" 0 0 0"/>
       <geometry>
         <box size=".4 .2 .1"/>
@@ -27,28 +30,29 @@
     </collision>
     <visual name='base_link_visual'>
-      <origin xyz="0 0 0" rpy="0 0 0"/>
+      <origin xyz="0 0 0" rpy=" 0 0 0"/>
       <geometry>
         <!--box size=".4 .2 .1"/-->
         <mesh filename = "package://bme_gazebo_basics/meshes/mogi_bot.dae"/>
       </geometry>
-      <material name="green"/>
-    </visual>
-  </link>
-    <joint type="continuous" name="front_left_wheel_joint">
+      <material name="orange"/>
+    </visual>
+  </link>
+  <!-- STEP 2 - Wheels -->
+  <joint type="continuous" name="front_left_wheel_joint">
     <origin xyz="0.15 0.15 0" rpy="0 0 0"/>
     <child link="front_left_wheel"/>
     <parent link="base_link"/>
     <axis xyz="0 1 0" rpy="0 0 0"/>
-    <limit effort="10000" velocity="1000"/> <!-- effort: torque limit ...-->
+    <limit effort="10000" velocity="1000"/>
     <dynamics damping="1.0" friction="1.0"/>
   </joint>
   <link name='front_left_wheel'>
     <inertial>
-      <mass value="5.0"/>
-      <origin xyz="0 0 0" rpy="0 1.5707 1.5707"/>
-      <inertia
-          ixx="0.1" ixy="0" ixz="0"
-          iyy="0.1" iyz="0"
-          izz="0.1"
+      <mass value="0.5"/>
+      <origin xyz="0 0 0" rpy="0 1.5707 1.5707"/>
+      <inertia
+          ixx="0.001354166" ixy="0" ixz="0"
+          iyy="0.001354166" iyz="0"
+          izz="0.0025"
       />
     </inertial>
@@ -62,37 +66,8 @@
       <origin xyz="0 0 0" rpy="0 1.5707 1.5707"/>
       <geometry>
-        <mesh filename = "package://bme_gazebo_basics/meshes/wheel.dae"/>
-      </geometry>
-    </visual>
-  </link>
-    <joint type="continuous" name="rear_left_wheel_joint">
-    <origin xyz="-0.15 0.15 0" rpy="0 0 0"/>
-    <child link="rear_left_wheel"/>
-    <parent link="base_link"/>
-    <axis xyz="0 1 0" rpy="0 0 0"/>
-    <limit effort="10000" velocity="1000"/> <!-- effort: torque limit ...-->
-    <dynamics damping="1.0" friction="1.0"/>
-  </joint>
-  <link name='rear_left_wheel'>
-    <inertial>
-      <mass value="5.0"/>
-      <origin xyz="0 0 0" rpy="0 1.5707 1.5707"/>
-      <inertia
-          ixx="0.1" ixy="0" ixz="0"
-          iyy="0.1" iyz="0"
-          izz="0.1"
-      />
-    </inertial>
-    <collision name='collision'>
-      <origin xyz="0 0 0" rpy="0 1.5707 1.5707"/>
-      <geometry>
-        <cylinder radius=".1" length=".05"/>
-      </geometry>
-    </collision>
-    <visual name='rear_left_wheel_visual'>
-      <origin xyz="0 0 0" rpy="0 1.5707 1.5707"/>
-      <geometry>
-        <mesh filename = "package://bme_gazebo_basics/meshes/wheel.dae"/>
-      </geometry>
+        <!--cylinder radius=".1" length=".05"/-->
+        <mesh filename = "package://bme_gazebo_basics/meshes/wheel.dae"/>
+      </geometry>
+      <material name="green"/>
     </visual>
   </link>
@@ -107,10 +82,10 @@
   <link name='front_right_wheel'>
     <inertial>
-      <mass value="5.0"/>
-      <origin xyz="0 0 0" rpy="0 1.5707 1.5707"/>
-      <inertia
-          ixx="0.1" ixy="0" ixz="0"
-          iyy="0.1" iyz="0"
-          izz="0.1"
+      <mass value="0.5"/>
+      <origin xyz="0 0 0" rpy="0 1.5707 1.5707"/>
+      <inertia
+          ixx="0.001354166" ixy="0" ixz="0"
+          iyy="0.001354166" iyz="0"
+          izz="0.0025"
       />
     </inertial>
@@ -124,9 +99,44 @@
       <origin xyz="0 0 0" rpy="0 1.5707 1.5707"/>
       <geometry>
-        <mesh filename = "package://bme_gazebo_basics/meshes/wheel.dae"/>
-      </geometry>
-    </visual>
-  </link>
-    <joint type="continuous" name="rear_right_wheel_joint">
+        <!--cylinder radius=".1" length=".05"/-->
+        <mesh filename = "package://bme_gazebo_basics/meshes/wheel.dae"/>
+      </geometry>
+      <material name="green"/>
+    </visual>
+  </link>
+  <joint type="continuous" name="rear_left_wheel_joint">
+    <origin xyz="-0.15 0.15 0" rpy="0 0 0"/>
+    <child link="rear_left_wheel"/>
+    <parent link="base_link"/>
+    <axis xyz="0 1 0" rpy="0 0 0"/>
+    <limit effort="10000" velocity="1000"/>
+    <dynamics damping="1.0" friction="1.0"/>
+  </joint>
+  <link name='rear_left_wheel'>
+    <inertial>
+      <mass value="0.5"/>
+      <origin xyz="0 0 0" rpy="0 1.5707 1.5707"/>
+      <inertia
+          ixx="0.001354166" ixy="0" ixz="0"
+          iyy="0.001354166" iyz="0"
+          izz="0.0025"
+      />
+    </inertial>
+    <collision name='collision'>
+      <origin xyz="0 0 0" rpy="0 1.5707 1.5707"/>
+      <geometry>
+        <cylinder radius=".1" length=".05"/>
+      </geometry>
+    </collision>
+    <visual name='rear_left_wheel_visual'>
+      <origin xyz="0 0 0" rpy="0 1.5707 1.5707"/>
+      <geometry>
+        <!--cylinder radius=".1" length=".05"/-->
+        <mesh filename = "package://bme_gazebo_basics/meshes/wheel.dae"/>
+      </geometry>
+      <material name="green"/>
+    </visual>
+  </link>
+  <joint type="continuous" name="rear_right_wheel_joint">
     <origin xyz="-0.15 -0.15 0" rpy="0 0 0"/>
     <child link="rear_right_wheel"/>
@@ -138,10 +148,10 @@
   <link name='rear_right_wheel'>
     <inertial>
-      <mass value="5.0"/>
-      <origin xyz="0 0 0" rpy="0 1.5707 1.5707"/>
-      <inertia
-          ixx="0.1" ixy="0" ixz="0"
-          iyy="0.1" iyz="0"
-          izz="0.1"
+      <mass value="0.5"/>
+      <origin xyz="0 0 0" rpy="0 1.5707 1.5707"/>
+      <inertia
+          ixx="0.001354166" ixy="0" ixz="0"
+          iyy="0.001354166" iyz="0"
+          izz="0.0025"
       />
     </inertial>
@@ -155,7 +165,50 @@
       <origin xyz="0 0 0" rpy="0 1.5707 1.5707"/>
       <geometry>
-        <mesh filename = "package://bme_gazebo_basics/meshes/wheel.dae"/>
-      </geometry>
-    </visual>
-  </link>
+        <!--cylinder radius=".1" length=".05"/-->
+        <mesh filename = "package://bme_gazebo_basics/meshes/wheel.dae"/>
+      </geometry>
+      <material name="green"/>
+    </visual>
+  </link>
+  <!-- STEP 4 - Gazebo physics -->
+  <gazebo reference="front_left_wheel">
+    <!-- kp and kd for rubber -->
+    <kp>1000000.0</kp>
+    <kd>100.0</kd>
+    <mu1>1.5</mu1>
+    <mu2>1.5</mu2>
+    <fdir1>1 0 0</fdir1>
+    <maxVel>1.0</maxVel>
+    <minDepth>0.00</minDepth>
+  </gazebo>
+  <gazebo reference="front_right_wheel">
+    <!-- kp and kd for rubber -->
+    <kp>1000000.0</kp>
+    <kd>100.0</kd>
+    <mu1>1.5</mu1>
+    <mu2>1.5</mu2>
+    <fdir1>1 0 0</fdir1>
+    <maxVel>1.0</maxVel>
+    <minDepth>0.00</minDepth>
+  </gazebo>
+  <gazebo reference="rear_left_wheel">
+    <!-- kp and kd for rubber -->
+    <kp>1000000.0</kp>
+    <kd>100.0</kd>
+    <mu1>1.5</mu1>
+    <mu2>1.5</mu2>
+    <fdir1>1 0 0</fdir1>
+    <maxVel>1.0</maxVel>
+    <minDepth>0.00</minDepth>
+  </gazebo>
+  <gazebo reference="rear_right_wheel">
+    <!-- kp and kd for rubber -->
+    <kp>1000000.0</kp>
+    <kd>100.0</kd>
+    <mu1>1.5</mu1>
+    <mu2>1.5</mu2>
+    <fdir1>1 0 0</fdir1>
+    <maxVel>1.0</maxVel>
+    <minDepth>0.00</minDepth>
+  </gazebo>
 </robot>
